Commit message: feat: update launch and URDF files for improved robot description configuration

File: description_launch/urdf/questix.xacro (robot description, xacro)
@@ -2,5 +2,5 @@
   <xacro:property name="side" value="0.5" />
     <!-- questix-->
-    <!--<link name="base_link">
+    <link name="base_link">
     <visual>
       <origin xyz="0 0 0.1" rpy="0 0 0"/>
@@ -9,7 +9,7 @@
       </geometry>
     </visual>
-    </link>-->
+    </link>
     <!-- test用の箱表示 -->
-    <link name="base_link">
+    <!--<link name="base_link">
       <visual>
         <origin xyz="0 0 0" rpy="0 0 0"/>
@@ -18,4 +18,4 @@
         </geometry>
       </visual>
-    </link>
+    </link>-->
 </robot>
